Commit message: Added RSP launch file

File: description/robot.urdf.xacro (robot description, xacro)
@@ -1,4 +1,3 @@
 <?xml version="1.0"?>
 <robot xmlns:xacro="http://www.ros.org/wiki/xacro"  name="robot">
-    <xacro:include filename="rover_core.xacro"/>
 </robot>

File: description/rover.urdf.xacro (robot description, xacro)
@@ -1,4 +1,4 @@
 <?xml version="1.0"?>
-<robot xmlns:xacro="http://www.ros.org/wiki/xacro"  name="robot">
-    <xacro:include filename="rover_core.xacro"/>
+<robot xmlns:xacro="http://ros.org/wiki/xacro" name="my_robot">
+    <xacro:include filename="rover_core.xacro" />
 </robot>

File: description/rover_core.xacro (robot description, xacro)
@@ -1,4 +1,10 @@
 <?xml version="1.0"?>
-<robot xmlns:xacro="http://www.ros.org/wiki/xacro"  name="robot">
-    <link name="base_link"></link>
+<robot xmlns:xacro="http://www.ros.org/wiki/xacro" >
+    <link name="base_link">
+        <visual>
+            <geometry>
+                <box size="1 1 1"/>
+            </geometry>
+        </visual>
+    </link>
 </robot>
