Commit message: updated rover

File: src/description/vicharaka-rover.urdf (robot description, URDF)
Before this commit: robot vicharaka_rover, 23 links, 22 joints
Links:
- removed link lidar
- added link laser_frame; collision cylinder length=0.04 radius=0.05; visual cylinder length=0.04 radius=0.05
Joints:
- removed joint base_lidar_joint
- added joint laser_joint: type fixed, parent base_link, child laser_frame, origin xyz=0.122 0 0.212 rpy=0 0 0

Commit message: added depth camera and imu files

File: src/description/vicharaka-rover.urdf (robot description, URDF)
Before this commit: robot vicharaka-rover, 23 links, 22 joints
Links:
- added link camera_link; visual box size=0.010 0.03 0.03
Joints:
- added joint camera_joint: type fixed, parent base_link, child camera_link, origin xyz=0.305 0 0.08 rpy=0 0 0

Commit message: update urdf

File: src/description/vicharaka-rover.urdf (robot description, URDF)
Before this commit: robot vicharaka-rover, 24 links, 23 joints
Links:
- added link antenna_link; visual cylinder length=0.6 radius=0.015
- link camera_link: geometry visual box size=0.025 0.12 0.03
Joints:
- removed joint base_joint
- added joint antenna_joint: type fixed, parent base_link, child antenna_link, origin xyz=-0.305 0 0 rpy=0 0 0
- added joint base_footprint_joint: type fixed, parent base_link, child base_footprint, origin xyz=0 0 0 rpy=0 0 0

Commit message: added ponitcloud conversion file

File: src/description/vicharaka-rover.urdf (robot description, URDF)
Before this commit: robot vicharaka-rover, 25 links, 24 joints
Links:
- added link chassis; visual box size=0.6 0.4 0.2
- link base_link: geometry 
Joints:
- added joint chassis_joint: type fixed, parent base_link, child chassis, origin xyz=0 0 0 rpy=0 0 0
- joint base_footprint_joint: child base_footprint -> base_link; origin xyz=0 0 0 rpy=0 0 0 -> xyz=0 0 0.5 rpy=0 0 0; parent base_link -> base_footprint

Commit message: added global localisation config

File: src/description/vicharaka-rover.urdf (robot description, URDF)
Before this commit: robot vicharaka-rover, 26 links, 25 joints
Links:
- removed link chassis
- link base_link: geometry visual box size=0.6 0.4 0.2
Joints:
- removed joint chassis_joint
- joint base_footprint_joint: origin xyz=0 0 0.5 rpy=0 0 0 -> xyz=0 0 0 rpy=0 0 0
- joint laser_joint: origin xyz=0.122 0 0.212 rpy=0 0 0 -> xyz=-0.187 0 0.212 rpy=0 0 0
